File: geiger.brd (EAGLE design)
At the start: 148.6 x 81.3 mm, 46 parts, among them IC1 LM4041A12DBZ, IC2 MAX4105EUK, IC3 74LS14D, IC5 REG1118, Q1 N-HEXFET-2D_SOT232-IRLL2705

Commit message: Up to date with built Rev1
Parts:
- removed G1: AB9V, battery:AB9V
- removed IC5: REG1118, burr-brown:SOT223
- added C18: 1000uF, rcl:TT5D10
- added C19: 1uf, rcl:C0603
- added U$1, U$2, U$3, U$5: BINDING-POST, geiger:BINDING-POST
- C1: value (none) -> 100pF
- C10, C11, C12, C13, C14, C15, C16, C2, C3, C4, C5, C6, C7, C8, C9: value (none) -> 0.1uF
- C17: value (none) -> 1uf
- IC1: value LM4041A12DBZ -> 2.5V
- L1: value (none) -> 4.7uH
- R1: value (none) -> 750k
- R2: value (none) -> 100k
- R3: value (none) -> 10k
- R4: value (none) -> 68M
- R5: value (none) -> 2M
- R6: value (none) -> 500k
- moved D1 22.9 mm to (25.9, 14.0)
- moved C1 21.9 mm to (40.4, 16.3)
- moved C17 21.9 mm to (32.0, 10.4)
- moved C2 21.9 mm to (22.6, 18.5)
- moved IC1 21.9 mm to (39.4, 12.2)
- moved L1 21.9 mm to (16.3, 16.0)
- moved Q1 21.9 mm to (18.8, 6.60)
- moved R1 21.9 mm to (38.4, 16.3)
- moved R2 21.9 mm to (36.3, 16.3)
- moved R3 21.9 mm to (34.3, 16.3)
- moved R4 21.9 mm to (31.8, 19.6)
- moved R5 21.9 mm to (31.8, 16.8)
- moved IC3 21.9 mm to (27.2, 7.87)
- moved R6 21.9 mm to (26.7, 19.1)
- moved IC2 21.8 mm to (35.8, 12.2)
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Connections:
- net N$19 renamed +HV
- removed net N$20: C16.2, D16.C
- removed net N$9: G1.+, IC5.3
- new net HV: C16.2, D16.C, U$5.P$1
- net GND: now also C18.-, C19.1, U$1.P$1, U$3.P$1; no longer G1.-, IC5.2
- net VCC: now also C18.+, C19.2, U$2.P$1; no longer IC5.1
Routing:
- net VCC: track 62.1 -> 81.3 mm
- net N$9: track 17.0 -> 0.00 mm
- net HV: track 0.00 -> 11.8 mm
- net GND: track 0.00 -> 8.78 mm, vias 0 -> 2
- net N$24: track 51.0 -> 43.2 mm
- net N$7: track 41.4 -> 37.3 mm
- net N$20: track 2.71 -> 0.00 mm
- net N$2: track 3.90 -> 6.01 mm
- net N$4: track 25.8 -> 23.7 mm
- net N$5: track 20.3 -> 20.8 mm
- added copper zone on layer 1, net GND
- added copper zone on layer 16, net GND
Other:
- board size 148.6 x 81.3 mm -> 61 x 45.7 mm
- board text added: "+5V"
- board text added: "+HV"
- board text added: "2016/09/11"
- board text added: "GND"
- board text added: "High Voltage Step-Up Converter"
